File: vibrador/VIbrador.sch (KiCad schematic (older format))
At the start: 6 parts, among them U1 Pila3,7V, U3 Buzzer, U4 HC-05, U5 Buzzer, U6 PiZeroW

Commit message: Esquematico
Parts:
- added U2: StepDown, VibradorPCB:StepDown, symbol VIbrador-rescue:StepDown
- added U7: Pila3,7V-Modulos-VIbrador-rescue, VibradorPCB:Pila de Litio, symbol VIbrador-rescue:Pila3,7V-Modulos-VIbrador-rescue
- A1: symbol MCU_Module:Arduino_Nano_v3.x -> VIbrador-rescue:Arduino_Nano_v3.x-MCU_Module
Connections:
- net labels added: IN+, IN-, OUT+, OUT-, Rx_Rasp, Rx_rasp, Tx_rasp
- wire segments 44 -> 85
Other:
- moved on the sheet: U1
Changed lines of the file:
@@
 EESchema Schematic File Version 4
-LIBS:VIbrador-cache
-EELAYER 29 0
+EELAYER 30 0
 EELAYER END
 $Descr A4 8268 11693 portrait
@@
 L VIbrador-rescue:Pila3,7V-Modulos-VIbrador-rescue U1
 U 1 1 5E6ECDF3
-P 4650 2300
-F 0 "U1" H 4700 2515 50  0000 C CNN
-F 1 "Pila3,7V" H 4700 2424 50  0000 C CNN
-F 2 "VibradorPCB:Pila de Litio" H 4650 2300 50  0001 C CNN
-F 3 "" H 4650 2300 50  0001 C CNN
-	1    4650 2300
-	1    0    0    -1
-$EndComp
-Text GLabel 4350 2500 3    50   Input ~ 0
-VIN
-Text GLabel 5050 2500 3    50   Input ~ 0
-GND
-Wire Wire Line
-	5050 2500 5050 2350
-Wire Wire Line
-	5050 2350 4950 2350
+P 4750 2400
+F 0 "U1" H 4800 2615 50  0000 C CNN
+F 1 "Pila3,7V" H 4800 2200 50  0000 C CNN
+F 2 "VibradorPCB:Pila de Litio" H 4750 2400 50  0001 C CNN
+F 3 "" H 4750 2400 50  0001 C CNN
+	1    4750 2400
+	-1   0    0    1
+$EndComp
 Wire Wire Line
 	4450 2350 4350 2350
-Wire Wire Line
-	4350 2350 4350 2500
-Text GLabel 2750 1350 2    50   Input ~ 0
-VIN
-Text GLabel 2950 3800 0    50   Input ~ 0
-GND
 Text GLabel 4500 4800 3    50   Input ~ 0
 TX
@@
 $EndComp
 $Comp
-L MCU_Module:Arduino_Nano_v3.x A1
+L VIbrador-rescue:Arduino_Nano_v3.x-MCU_Module A1
 U 1 1 5E91EE2F
 P 2850 2500
@@
 Wire Wire Line
 	2750 1350 2750 1500
+$Comp
+L VIbrador-rescue:Pila3,7V-Modulos-VIbrador-rescue U7
+U 1 1 5E94B3CF
+P 5750 2400
+F 0 "U7" H 5800 2615 50  0000 C CNN
+F 1 "Pila3,7V-Modulos-VIbrador-rescue" H 5800 2200 50  0000 C CNN
+F 2 "VibradorPCB:Pila de Litio" H 5750 2400 50  0001 C CNN
+F 3 "" H 5750 2400 50  0001 C CNN
+	1    5750 2400
+	-1   0    0    1
+$EndComp
+Wire Wire Line
+	5050 2350 4950 2350
+Wire Wire Line
+	5450 2350 5350 2350
+Wire Wire Line
+	5350 2350 5350 2450
+Wire Wire Line
+	5350 2450 5050 2450
+Wire Wire Line
+	5050 2450 5050 2350
+$Comp
+L VIbrador-rescue:StepDown U2
+U 1 1 5E9524F1
+P 5250 2800
+F 0 "U2" H 5275 3075 50  0000 C CNN
+F 1 "StepDown" H 5275 2984 50  0000 C CNN
+F 2 "VibradorPCB:StepDown" H 5250 2800 50  0001 C CNN
+F 3 "" H 5250 2800 50  0001 C CNN
+	1    5250 2800
+	1    0    0    -1
+$EndComp
+Text GLabel 4800 2850 0    50   Input ~ 0
+IN+
+Text GLabel 6250 2350 2    50   Input ~ 0
+IN+
+Text GLabel 4200 2350 0    50   Input ~ 0
+IN-
+Text GLabel 4800 3050 0    50   Input ~ 0
+IN-
+Wire Wire Line
+	4800 2850 4850 2850
+Wire Wire Line
+	4850 2850 4850 2750
+Wire Wire Line
+	4850 2750 5050 2750
+Wire Wire Line
+	4800 3050 4850 3050
+Wire Wire Line
+	4850 3050 4850 3150
+Wire Wire Line
+	4850 3150 5050 3150
+Wire Wire Line
+	4350 2350 4350 2450
+Wire Wire Line
+	4350 2450 4200 2450
+Wire Wire Line
+	4200 2450 4200 2350
+Wire Wire Line
+	5950 2350 6050 2350
+Wire Wire Line
+	6050 2350 6050 2450
+Wire Wire Line
+	6050 2450 6250 2450
+Wire Wire Line
+	6250 2450 6250 2350
+Text GLabel 5800 2850 2    50   Input ~ 0
+OUT+
+Text GLabel 5800 3050 2    50   Input ~ 0
+OUT-
+Wire Wire Line
+	5800 2850 5650 2850
+Wire Wire Line
+	5650 2850 5650 2750
+Wire Wire Line
+	5650 2750 5450 2750
+Wire Wire Line
+	5450 3150 5650 3150
+Wire Wire Line
+	5650 3150 5650 3050
+Wire Wire Line
+	5650 3050 5800 3050
+Text GLabel 2350 2100 0    50   Input ~ 0
+Tx_rasp
+Text GLabel 2350 2200 0    50   Input ~ 0
+Rx_Rasp
+Text GLabel 3850 4650 2    50   Input ~ 0
+Tx_rasp
+Text GLabel 3850 4750 2    50   Input ~ 0
+Rx_rasp
+Wire Wire Line
+	3850 4650 3750 4650
+Wire Wire Line
+	3750 4650 3750 4600
+Wire Wire Line
+	3750 4600 3400 4600
+Wire Wire Line
+	3400 4600 3400 4650
+Wire Wire Line
+	3400 4650 3200 4650
+Wire Wire Line
+	3850 4750 3750 4750
+Wire Wire Line
+	3750 4750 3750 4700
+Wire Wire Line
+	3750 4700 3400 4700
+Wire Wire Line
+	3400 4700 3400 4750
+Wire Wire Line
+	3400 4750 3200 4750
+Text GLabel 3700 4350 2    50   Input ~ 0
+OUT+
+Wire Wire Line
+	3600 4350 3600 4300
+Wire Wire Line
+	3600 4300 3400 4300
+Wire Wire Line
+	3400 4300 3400 4350
+Wire Wire Line
+	3400 4350 3200 4350
+Text GLabel 3750 5250 2    50   Input ~ 0
+OUT-
+Wire Wire Line
+	3600 5250 3600 5300
+Wire Wire Line
+	3600 5300 3400 5300
+Wire Wire Line
+	3400 5300 3400 5250
+Wire Wire Line
+	3400 5250 3200 5250
+Wire Wire Line
+	3700 4350 3600 4350
+Wire Wire Line
+	3600 5250 3750 5250
 $EndSCHEMATC
