File: vibrador/VIbrador.kicad_pcb (KiCad board)
At the start: 2 copper layers, 8 parts, among them U1 Pila3,7V, U2 StepDown, U3 Buzzer, U4 HC-05, U5 Buzzer, U6 PiZeroW

Commit message: Se finalizo PCB
Se cambio la huella de pila, y posicion de rx y tx en arduino
Parts:
- removed the U1 at (133.6, 178.4)
- removed the U1 at (134.4, 157.1)
- added U1: Pila3,7V, VibradorPCB:Pila de Litio, F.Cu at (57.1, 177.7)
- added U7: Pila3,7V-Modulos-VIbrador-rescue, VibradorPCB:Pila de Litio, F.Cu at (135.1, 158.0)
- moved U5 10.9 mm to (70.3, 141.2), turned to 90 degrees
- moved U3 2.84 mm to (122.0, 141.1)
Connections:
- A1 pad 13: TX -> RX
- A1 pad 14: RX -> TX
- A1 pad 29: GND -> OUT-
- A1 pad 30: VIN -> OUT+
- A1 pad 4: GND -> OUT-
- A1 pad 5: Net-(A1-Pad5) -> Tx_rasp
- A1 pad 6: Net-(A1-Pad6) -> Rx_rasp
- U3 pad 2: GND -> OUT-
- U4 pad 2: VIN -> OUT+
- U4 pad 3: GND -> OUT-
- U5 pad 2: GND -> OUT-
- U6 pad 10: Net-(U6-Pad10) -> Rx_rasp
- U6 pad 2: Net-(U6-Pad2) -> OUT+
- U6 pad 20: Net-(U6-Pad20) -> OUT-
- U6 pad 8: Net-(U6-Pad8) -> Tx_rasp
Routing:
- net OUT-: track 0.00 -> 300.4 mm
- net OUT+: track 0.00 -> 144.3 mm
- net D9: track 0.00 -> 87.6 mm
- net Tx_rasp: track 0.00 -> 79.6 mm
- net Rx_rasp: track 0.00 -> 79.3 mm
- net IN-: track 0.00 -> 76.1 mm
- net RX: track 0.00 -> 52.9 mm
- net IN+: track 0.00 -> 51.9 mm
- net TX: track 0.00 -> 49.3 mm
- net Net-(U1-Pad1): track 0.00 -> 19.7 mm
- added copper zone on B.Cu, net OUT-

Commit message: Se unieron IN- Y OUT- ya que los dos son GND de el step down y es lo mismo
Parts:
- moved U1 6.18 mm to (56.4, 183.8)
- moved U2 6.18 mm to (95.4, 128.9)
- moved U5 6.18 mm to (69.6, 147.3)
- moved U7 6.18 mm to (134.4, 164.1)
- moved A1 6.18 mm to (127.6, 133.4)
- moved U4 6.18 mm to (121.0, 50.2)
- moved U6 6.18 mm to (85.4, 124.3)
- moved U3 6.18 mm to (121.3, 147.2)
Connections:
- A1 pad 29: OUT- -> IN-
- A1 pad 4: OUT- -> IN-
- U2 pad 4: OUT- -> IN-
- U3 pad 2: OUT- -> IN-
- U4 pad 3: OUT- -> IN-
- U5 pad 2: OUT- -> IN-
- U6 pad 20: OUT- -> IN-
Routing:
- net OUT-: track 300.4 -> 0.00 mm
- net IN-: track 76.1 -> 376.5 mm
- added copper zone on B.Cu, net IN-
- removed copper zone on B.Cu, net OUT-

Commit message: Se termino el case falta hacerle el hueco dela bateria
Connections:
- A1 pad 13: RX -> Net-(A1-Pad13)
- A1 pad 14: TX -> Net-(A1-Pad14)
- U6 pad 16: Net-(U6-Pad16) -> TX
- U6 pad 18: Net-(U6-Pad18) -> RX
Routing:
- net TX: track 49.3 -> 81.3 mm
- net RX: track 52.9 -> 67.3 mm
- net Tx_rasp: track 79.6 -> 85.3 mm
- net Rx_rasp: track 79.3 -> 84.7 mm
- net IN-: track 376.5 -> 377.1 mm
